File: hardware/disappointment.kicad_pcb (KiCad board)
At the start: 2 copper layers, 175.3 x 58.4 mm, 70 parts, among them J1 Bus_ISA_16bit, J2 Conn_01x02_Pin, J3 Conn_02x10_Odd_Even, J5 ATX-24, U1 F85226AF, U2 L7905

Commit message: cleanups
Parts:
- moved ? 2.54 mm to (213.9, 83.4)
- moved ? 2.54 mm to (69.2, 83.4)
- moved D5 1.29 mm to (84.4, 110.5)
- moved D1 0.53 mm to (100.9, 110.5)
- moved D3 0.43 mm to (117.4, 110.5)
- moved D2 0.41 mm to (109.2, 110.5)
- moved D4 0.33 mm to (92.7, 110.5)
Routing:
- net Net-(D5-K): track 9.82 -> 11.2 mm
Other:
- board size 175.3 x 58.4 mm -> 170 x 58.4 mm

Commit message: what a... letdown?
Routing:
- net /SMEMR#: track 93.1 -> 94.3 mm
- net /SA7: track 66.6 -> 67.5 mm
- net +3.3V: track 210.8 -> 210.0 mm
- net /SA3: track 66.5 -> 65.8 mm
- net /SA2: track 67.0 -> 66.5 mm
- net /SA0: track 66.6 -> 66.1 mm
- net GND: vias 63 -> 69
Other:
- board text added: "github/rasteri/dISAppointment"
- board text added: "v0.2"
- board text removed: "RASTERI.COM -- v0.2"

Commit message: added the correct resistors
Parts:
- removed R3, R4: 8.2K, Resistor_SMD:R_1206_3216Metric_Pad1.30x1.75mm_HandSolder
- added R17: 1K, Resistor_SMD:R_1206_3216Metric_Pad1.30x1.75mm_HandSolder, F.Cu at (116.4, 122.5)
- added R18: 1K, Resistor_SMD:R_1206_3216Metric_Pad1.30x1.75mm_HandSolder, F.Cu at (113.1, 122.5)
- added R19: 1K, Resistor_SMD:R_1206_3216Metric_Pad1.30x1.75mm_HandSolder, F.Cu at (109.3, 122.5)
- J2: value Conn_01x02_Pin -> PS_ON
- J3: value Conn_02x10_Odd_Even -> LPC
- RN18: value 1K -> 8.2K
- moved RN18 13.1 mm to (95.7, 124.3), turned to 90 degrees
- moved R8 7.28 mm to (102.2, 115.6), turned to 90 degrees
- moved RN12 3.96 mm to (95.1, 114.6)
- moved RN5 3.96 mm to (99.0, 114.6)
- moved C19 2.85 mm to (102.5, 99.0), turned to -90 degrees
- moved C18 2.83 mm to (112.5, 99.0), turned to -90 degrees
- moved RN17 2.18 mm to (120.0, 123.1)
- moved C15 1.62 mm to (80.0, 99.0), turned to -90 degrees
- moved D1 1.45 mm to (100.9, 109.0)
- moved D2 1.45 mm to (109.2, 109.0)
- moved D3 1.45 mm to (117.4, 109.0)
- moved D4 1.45 mm to (92.7, 109.0)
- moved C17 0.29 mm to (92.0, 99.0)
Connections:
- RN16 pad 1: /DRQ0 -> /DRQ5
- RN16 pad 2: /DRQ5 -> /DRQ6
- RN16 pad 3: /DRQ6 -> /DRQ7
- RN16 pad 4: /DRQ7 -> /MASTER#
- RN16 pad 5: GND -> +5V
- RN18 pad 1: /SMEMR# -> unconnected-(RN18-R1.1-Pad1)
- RN18 pad 2: /SMEMW# -> +5V
- RN18 pad 4: /OWS# -> GND
- RN18 pad 5: +5V -> /DRQ2
- RN18 pad 6: +5V -> unconnected-(RN18-R3.2-Pad6)
- RN18 pad 7: +5V -> /IRQ9
- RN18 pad 8: +5V -> unconnected-(RN18-R1.2-Pad8)
- RN8 pad 4: unconnected-(RN8-R4.1-Pad4) -> /DRQ0
- RN8 pad 5: +5V -> GND
Routing:
- net +5V: track 561.3 -> 576.2 mm
- net /SD6: track 107.5 -> 117.1 mm
- net /SD7: track 111.1 -> 120.6 mm
- net /SD5: track 104.2 -> 113.5 mm
- net /SD4: track 100.4 -> 109.1 mm
- net /SD3: track 98.9 -> 107.1 mm
- net /SD2: track 89.6 -> 97.8 mm
- net /SD1: track 87.1 -> 95.1 mm
- net /IOR#: track 88.4 -> 96.2 mm
- net /SD0: track 88.0 -> 95.4 mm
- net +12V: track 45.5 -> 50.4 mm, vias 0 -> 1
- net -12V: track 76.7 -> 71.8 mm
- net /SMEMW#: track 95.3 -> 90.5 mm
- net /SMEMR#: track 94.3 -> 89.6 mm
- net /IOW#: track 86.8 -> 91.2 mm
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Other:
- board text added: "v0.3"
- board text removed: "v0.2"

Commit message: silkscreen cleanup
Parts:
- D1, D2, D3, D4, D5: footprint LED_SMD:LED_1206_3216Metric -> andy:LED_1206_3216Metric
Other:
- board size 170 x 58.4 mm -> 164.7 x 58.4 mm
- board text added: "v0.4"
- board text removed: "v0.3"
