File: hardware/disappointment.kicad_sch (KiCad schematic)
At the start: 63 parts, among them J1 Bus_ISA_16bit, J2 PS_ON, J3 LPC, J5 ATX-24, U1 F85226AF, U2 L7905

Commit message: silkscreen cleanup
Parts:
- D1, D2, D3, D4, D5: footprint LED_SMD:LED_1206_3216Metric -> andy:LED_1206_3216Metric
